File: Hardware/PCB/mini_hvac_0/mini_hvac_0.kicad_pcb (KiCad board)
At the start: 2 copper layers, 80 x 150 mm, 25 parts, among them J1 Conn_01x03_Pin, J10 Conn_01x03_Pin, J11 Conn_01x03_Pin, J12 Conn_01x03_Pin, J13 Conn_01x03_Pin, J14 Conn_01x04_Pin, J15 Conn_01x04_Socket, J16 Conn_01x02_Pin, J17 Conn_01x04_Pin, J2 Conn_01x03_Pin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

Commit message: final pcb, shrinked
Parts:
- moved SW1 5.55 mm to (170.2, 77.2)
- moved SW2 5.55 mm to (170.2, 67.5)
- moved SW3 5.55 mm to (170.2, 57.8)
- moved J8 5.01 mm to (172.5, 45.0)
Routing:
- net +5V: track 175.1 -> 209.5 mm
- net D4: track 60.7 -> 55.4 mm
- net D2: track 70.9 -> 66.4 mm
- net D3: track 64.9 -> 60.5 mm
- net D8: track 71.0 -> 73.4 mm
- added copper zone on B.Cu, net GND
- added copper zone on F.Cu, net GND
Other:
- board size 80 x 150 mm -> 81.5 x 54 mm
